File: Hardware/GeoFence.sch (KiCad schematic (older format))
At the start: 61 parts, among them J1 U.FL, J2 microB, J4 Qwiic_Connector, Q1 8/16/20MHz, U1 TITAN X1 GPS, U2 74LVC1G08SE, U3 CH340G, U4 MIC5205, U5 ATMEGA328, Y1 12MHz

Commit message: Finished Schematic
Got the rest of the EAGLE to KiCad conversions done and got everything
airwired properly (Hell is a real place called "CvPcb"). Beginnings of a
layout are happening now.
Parts:
- removed C5, C6: 10uF, EIA3216, symbol CAP_POL1206
- removed C7: 0.1uF, symbol C_Small
- removed J4: Qwiic_Connector, SPARKX_1X04_1MM_RA, symbol Qwiic_Connector
- removed J5: ~, SPARKFUN-CONNECTORS_1X01_NO_SILK, symbol SPARKFUN-CONNECTORS_CONN_01PTH_NO_SILK_YES_STOP
- removed J7: ~, SPARKFUN-CONNECTORS_1X05_NO_SILK, symbol SPARKFUN-CONNECTORS_CONN_05NO_SILK
- removed JP10, JP9: ~, 1X02, symbol M02PTH
- removed JP11, JP8: ~, 1X12, symbol M12PTH
- removed LOGO1: SFE_LOGO_NAME.1_INCH, SPARKFUN-AESTHETICS_SFE_LOGO_NAME_.1, symbol SPARKFUN-AESTHETICS_SFE_LOGO_NAME.1_INCH
- removed LOGO2: SFE_LOGO_FLAME.1_INCH, SPARKFUN-AESTHETICS_SFE_LOGO_FLAME_.1, symbol SPARKFUN-AESTHETICS_SFE_LOGO_FLAME.1_INCH
- removed U4: MIC5205, SOT23-5, symbol V_REG_LDOSMD
- added C15, C5: 4.7uF, Capacitors_SMD:C_0603, symbol SPARKFUN-CAPACITORS_4.7UF0603
- added C6: 1.0uF, Capacitors_SMD:C_0603, symbol SPARKFUN-CAPACITORS_1.0UF-0805-25V-_+80_-20%_
- added C7: 2.2uF, Capacitors_SMD:C_0603, symbol SPARKFUN-CAPACITORS_2.2UF-0603-10V-20%
- added D10: BAT20J, DiscreteSemi:SparkFun-DiscreteSemi-SOD-323, symbol SPARKFUN-DISCRETESEMI_DIODE-SCHOTTKY-BAT20J
- added D11: Yellow, LEDs:LED_0603, symbol SPARKFUN-LED_LED-YELLOW0603
- added D12: RED, LEDs:LED_0603, symbol SPARKFUN-LED_LED-RED0603
- added D6, D7, D8: Green, LEDs:LED_0603, symbol LED
- added D9: BLUE, LEDs:LED_0603, symbol SPARKFUN-LED_LED-BLUE0603-RESCUE-GeoFence
- added J3: AVR_SPI_PROG_3X2PTH, Connectors:2X3, symbol AVR_SPI_PROG_3X2PTH
- added J4, J5: CONN_04, Connectors:1X04, symbol CONN_04
- added J6: CONN_04X2, Connectors:2X4, symbol CONN_04X2
- added JP1, JP7: STAND-OFF, Hardware:STAND-OFF, symbol SPARKFUN_STAND-OFF
- added JP8: LiPo, Connectors:JST-2-PTH, symbol SPARKFUN-CONNECTORS_M02JST-PTH-2
- added Q2: 2.5A/30V, DiscreteSemi:SparkFun-DiscreteSemi-SOT23-3, symbol SPARKFUN-DISCRETESEMI_MOSFET-PCHANNELDMG2307L
- added R14: 330, Resistors_SMD:R_0603, symbol R_Small
- added R15: 470, Resistors_SMD:R_0603, symbol R_Small
- added R16: 10k, Resistors_SMD:R_0603, symbol SPARKFUN-RESISTORS_10KOHM-0603-1_10W-1%
- added R17: 2.0k, Resistors_SMD:R_0603, symbol SPARKFUN-RESISTORS_2.0KOHM1_10W5%_0603_
- added R19, R20: 1K, Resistors_SMD:R_0603, symbol SPARKFUN-RESISTORS_1KOHM-1_10W-1%_0603_
- added U4: AP2112K-3.3V, IC:SOT23-5, symbol SPARKFUN-POWERIC_V_REG_LDOSMD
- added U6: MCP73831, IC:SOT23-5, symbol SPARKFUN-POWERIC_MCP73831
- B1: footprint SPARKX_6.8MM_COIN_CELL -> SparkX:SparkX-6.8MM_COIN_CELL
- C1, C10, C11, C12, C13, C14, C2, C3, C4, C8, C9: footprint (none) -> Capacitors_SMD:C_0603
- D1: footprint SPARKFUN-LED_LED-0603 -> LEDs:LED_0603; symbol SPARKFUN-LED_LED-BLUE0603 -> SPARKFUN-LED_LED-BLUE0603-RESCUE-GeoFence
- D2: footprint SPARKFUN-DISCRETESEMI_SOD-323 -> DiscreteSemi:SparkFun-DiscreteSemi-SOD-323
- D3, D4: footprint SPARKFUN-LED_LED-0603 -> LEDs:LED_0603
- D5, LED1: footprint 0603-LED-ALT1 -> LEDs:LED_0603
- FB1, L1: footprint SPARKFUN-COILS_0603 -> Inductors_SMD:L_0603
- J1: footprint SPARKX_U.FL -> SparkX:SparkX-U.FL
- J2: footprint (none) -> Connectors:USB-B-MICRO-SMD
- JP2, JP6: footprint SPARKFUN_MICRO-FIDUCIAL -> Aesthetics:FIDUCIAL-MICRO
- JP3, JP4: footprint SPARKFUN_STAND-OFF -> Hardware:STAND-OFF
- JP5: footprint SPARKFUN-JUMPERS_SMT-JUMPER_2_NC_TRACE_NO-SILK -> Jumpers:SMT-JUMPER_2_NC_TRACE_NO-SILK
- Q1: footprint RESONATOR-SMD-1:1 -> Clocks:RESONATOR-SMD-3.2X1.3
- R1: footprint SPARKFUN-RESISTORS_0603-RES -> Resistors_SMD:R_0603
- R10, R11: value 470 -> 330; footprint (none) -> Resistors_SMD:R_0603
- R12, R13, R2, R3, R4, R5, R6, R7, R8, R9: footprint (none) -> Resistors_SMD:R_0603
- S1: footprint (none) -> Switches:TACTILE_SWITCH_SMD_5.2MM
- U$1: footprint SPARKX_SPARKX-LARGE -> SparkX:SparkX-SPARKX-LARGE
- U1: footprint SPARKX_TITAN_X1_GPS -> SparkX:SparkX-TITAN_X1_GPS
- U2: footprint SERIAL-BASIC_SOT353 -> IC:SOT353
- U3: footprint SPARKFUN-DIGITALIC_SO016 -> IC:SO16
- U5: footprint TQFP32-08 -> IC:TQFP32-08
- Y1: footprint (none) -> Clocks:CRYSTAL-SMD-3.2X2.5MM
Connections:
- net labels added: ATRESET, STATUS, V_BATT, Z1Pin, Z2Pin, Z3Pin, Z4Pin
- net labels removed: D6, RAW, RESET, RX, TX
- wire segments 218 -> 221
Other:
- note added: "600mA out\n6V max in"
- note added: "ATmega328"
- note added: "Charge current:\nI_CHG = 1000 / R_PROG\nR_PROG=2k : I_CHG=500mA"
- note added: "GPIO\n"
- note added: "ISP Header\n"
- note added: "Lithium-Polymer Battery Charger (1-cell)"
- note added: "Power LED"
- note added: "Status LED"
- note added: "V_BATT should be a single-\ncell LiPo battery."
- note added: "Voltage Regulator and Battery Charger"
- note added: "Zone Status Pins"
- note removed: "3.3V Regulation"
- note removed: "Add ISP header"
- note removed: "LEDs"
- note removed: "Max Current Output: 150mA"
- note removed: "Max Voltage Input: 16VDC"
- note removed: "N. Seidle"
- note removed: "Resonator"
- note removed: "X10"
- moved on the sheet: B1, C1, C10, C11, C12, C13, C14, C2, C3, C4, C8, C9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

Commit message: Moved Reference labels to drwg layer
The board layout is beginning to take form
Parts:
- removed JP1, JP3, JP4, JP7: STAND-OFF, Hardware:STAND-OFF, symbol SPARKFUN_STAND-OFF
- removed LED1: Red, LEDs:LED_0603, symbol LED
- removed R5: 10k, Resistors_SMD:R_0603, symbol R_Small
Connections:
- wire segments 221 -> 218
Other:
- note removed: "Power LED"
- moved on the sheet: D9, R15

Commit message: Routing
Started Routing
Connections:
- net labels removed: A4, A5, VCC
- wire segments 218 -> 219

Commit message: Design Review Changes
Parts:
- removed C15, C5: 4.7uF, Capacitors_SMD:C_0603, symbol SPARKFUN-CAPACITORS_4.7UF0603
- removed C6: 1.0uF, Capacitors_SMD:C_0603, symbol SPARKFUN-CAPACITORS_1.0UF-0805-25V-_+80_-20%_
- removed C7: 2.2uF, Capacitors_SMD:C_0603, symbol SPARKFUN-CAPACITORS_2.2UF-0603-10V-20%
- removed D1, D9: BLUE, LEDs:LED_0603, symbol SPARKFUN-LED_LED-BLUE0603-RESCUE-GeoFence
- removed D11: Yellow, LEDs:LED_0603, symbol SPARKFUN-LED_LED-YELLOW0603
- removed D12: RED, LEDs:LED_0603, symbol SPARKFUN-LED_LED-RED0603
- removed JP5: ~, Jumpers:SMT-JUMPER_2_NC_TRACE_NO-SILK, symbol SPARKFUN-JUMPERS_JUMPER-SMT_2_NC_TRACE_NO-SILK
- removed R1, R19, R20: 1K, Resistors_SMD:R_0603, symbol SPARKFUN-RESISTORS_1KOHM-1_10W-1%_0603_
- removed R16: 10k, Resistors_SMD:R_0603, symbol SPARKFUN-RESISTORS_10KOHM-0603-1_10W-1%
- removed R17: 2.0k, Resistors_SMD:R_0603, symbol SPARKFUN-RESISTORS_2.0KOHM1_10W5%_0603_
- removed U2: 74LVC1G08SE, IC:SOT353, symbol SERIAL-BASIC_7408
- added C15, C5: 4.7uF, Capacitors_SMD:C_0603, symbol C_Small
- added C6: 1.0uF, Capacitors_SMD:C_0603, symbol C_Small
- added C7: 2.2uF, Capacitors_SMD:C_0603, symbol C_Small
- added D1, D9: Blue, LEDs:LED_0603, symbol LED
- added D11: Yellow, LEDs:LED_0603, symbol LED
- added D12: Red, LEDs:LED_0603, symbol LED
- added H1, H2: STAND-OFF, Hardware:STAND-OFF, symbol STAND-OFF
- added R1, R17, R18: 1k, Resistors_SMD:R_0603, symbol R_Small
- added R16: 2.0k, Resistors_SMD:R_0603, symbol R_Small
- added R5: 10k, Resistors_SMD:R_0603, symbol R_Small
- D5, D6, D7, D8: value Green -> Blue
- JP8: footprint Connectors:JST-2-PTH -> Connectors:JST-2-SMD
- R10, R11, R14, R8: value 330 -> 470
Connections:
- net labels removed: D2, D3, Z1Pin, Z2Pin, Z3Pin, Z4Pin
- wire segments 219 -> 218
- no-connect marks 0 -> 1
Other:
- note added: "Pulse Per Second\nLED"
- note added: "Zone 1"
- note added: "Zone 2"
- note added: "Zone 3"
- note added: "Zone 4"
- note removed: "Buffer for RX LED"
- note removed: "Pulse Per Second LED"
- moved on the sheet: B1, C8, D2, D3, D5, D6, D7, D8, R10, R11, R14, R3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
