File: Hardware/Panel/GeoFence-panel.kicad_pcb (KiCad board)
At the start: 2 copper layers, 92.5 x 132.6 mm, 426 parts, among them J1 U.FL, J2 microB, J3 AVR_SPI_PROG_3X2PTH, J4 CONN_04, J5 CONN_04, J6 CONN_04X2, Q1 8/16/20MHz, Q2 2.5A/30V, U1 TITAN X1 GPS, U3 CH340G, U4 AP2112K-3.3V, U5 ATMEGA328, U6 MCP73831, Y1 12MHz

Commit message: Panel Update
Parts:
- removed the B1 at (163.7, 139.8)
- removed the B1 at (132.8, 139.8)
- removed the B1 at (101.8, 139.8)
- removed the B1 at (163.7, 73.3)
- removed the B1 at (132.8, 73.3)
- removed the C1 at (150.0, 112.6)
- removed the C1 at (119.0, 112.6)
- removed the C1 at (88.0, 112.6)
- removed the C1 at (150.0, 46.0)
- removed the C1 at (119.0, 46.0)
- removed the C10 at (138.4, 121.2)
- removed the C10 at (107.4, 121.2)
- removed the C10 at (76.5, 121.2)
- removed the C10 at (138.4, 54.6)
- removed the C10 at (107.4, 54.6)
- removed the C11 at (157.2, 121.2)
- removed the C11 at (126.2, 121.2)
- removed the C11 at (95.2, 121.2)
- removed the C11 at (157.2, 54.6)
- removed the C11 at (126.2, 54.6)
- removed the C12 at (143.3, 124.2)
- removed the C12 at (112.3, 124.2)
- removed the C12 at (81.3, 124.2)
- removed the C12 at (143.3, 57.7)
- removed the C12 at (112.3, 57.7)
- removed the C13 at (144.4, 142.2)
- removed the C13 at (113.4, 142.2)
- removed the C13 at (82.5, 142.2)
- removed the C13 at (144.4, 75.6)
- removed the C13 at (113.4, 75.6)
- removed the C14 at (146.6, 142.2)
- removed the C14 at (115.6, 142.2)
- removed the C14 at (84.7, 142.2)
- removed the C14 at (146.6, 75.6)
- removed the C14 at (115.6, 75.6)
- removed the C15 at (163.8, 113.7)
- removed the C15 at (132.8, 113.7)
- removed the C15 at (101.8, 113.7)
- removed the C15 at (163.8, 47.1)
- removed the C15 at (132.8, 47.1)
- removed the C2 at (150.0, 107.4)
- removed the C2 at (119.0, 107.4)
- removed the C2 at (88.0, 107.4)
- removed the C2 at (150.0, 40.9)
- removed the C2 at (119.0, 40.9)
- removed the C3 at (147.6, 114.7)
- removed the C3 at (116.6, 114.7)
- removed the C3 at (85.6, 114.7)
- removed the C3 at (147.6, 48.1)
- removed the C3 at (116.6, 48.1)
- removed the C4 at (147.4, 124.4)
- removed the C4 at (116.4, 124.4)
- removed the C4 at (85.5, 124.4)
- removed the C4 at (147.4, 57.8)
- removed the C4 at (116.4, 57.8)
- removed the C5 at (161.6, 113.7)
- removed the C5 at (130.6, 113.7)
- removed the C5 at (99.6, 113.7)
- removed the C5 at (161.6, 47.1)
- removed the C5 at (130.6, 47.1)
- removed the C6 at (165.6, 121.2)
- removed the C6 at (134.6, 121.2)
- removed the C6 at (103.6, 121.2)
- removed the C6 at (165.6, 54.6)
- removed the C6 at (134.6, 54.6)
- removed the C7 at (163.1, 118.1)
- removed the C7 at (132.1, 118.1)
- removed the C7 at (101.1, 118.1)
- removed the C7 at (163.1, 51.6)
- removed the C7 at (132.1, 51.6)
- removed the C8 at (149.6, 143.3)
- removed the C8 at (118.6, 143.3)
- removed the C8 at (87.6, 143.3)
- removed the C8 at (149.6, 76.7)
- removed the C8 at (118.6, 76.7)
- removed the C9 at (145.5, 121.2)
- removed the C9 at (114.6, 121.2)
- removed the C9 at (83.6, 121.2)
- removed the C9 at (145.5, 54.6)
- removed the C9 at (114.6, 54.6)
- removed the D1 at (156.8, 124.4)
- removed the D1 at (125.8, 124.4)
- removed the D1 at (94.8, 124.4)
- removed the D1 at (156.8, 57.8)
- removed the D1 at (125.8, 57.8)
- removed the D10 at (163.8, 109.9)
- removed the D10 at (132.8, 109.9)
- removed the D10 at (101.8, 109.9)
- removed the D10 at (163.8, 43.4)
- removed the D10 at (132.8, 43.4)
- removed the D11 at (159.0, 118.4)
- removed the D11 at (128.0, 118.4)
- removed the D11 at (97.0, 118.4)
- removed the D11 at (159.0, 51.8)
- removed the D11 at (128.0, 51.8)
- removed the D12 at (154.9, 118.4)
- removed the D12 at (124.0, 118.4)
- removed the D12 at (93.0, 118.4)
- removed the D12 at (154.9, 51.8)
- removed the D12 at (124.0, 51.8)
- removed the D2 at (161.8, 133.6)
- removed the D2 at (130.8, 133.6)
- removed the D2 at (99.8, 133.6)
- removed the D2 at (161.8, 67.1)
- removed the D2 at (130.8, 67.1)
- removed the D3 at (151.4, 118.4)
- removed the D3 at (120.4, 118.4)
- removed the D3 at (89.4, 118.4)
- removed the D3 at (151.4, 51.8)
- removed the D3 at (120.4, 51.8)
- removed the D4 at (147.5, 118.4)
- removed the D4 at (116.5, 118.4)
- removed the D4 at (85.6, 118.4)
- removed the D4 at (147.5, 51.8)
- removed the D4 at (116.5, 51.8)
- removed the D5 at (138.4, 155.0)
- removed the D5 at (107.4, 155.0)
- removed the D5 at (76.5, 155.0)
- removed the D5 at (138.4, 88.4)
- removed the D5 at (107.4, 88.4)
- removed the D6 at (141.0, 155.0)
- removed the D6 at (110.0, 155.0)
- removed the D6 at (79.0, 155.0)
- removed the D6 at (141.0, 88.4)
- removed the D6 at (110.0, 88.4)
- removed the D7 at (143.5, 154.9)
- removed the D7 at (112.5, 154.9)
- removed the D7 at (81.5, 154.9)
- removed the D7 at (143.5, 88.4)
- removed the D7 at (112.5, 88.4)
- removed the D8 at (146.1, 154.9)
- removed the D8 at (115.1, 154.9)
- removed the D8 at (84.1, 154.9)
- removed the D8 at (146.1, 88.4)
- removed the D8 at (115.1, 88.4)
- removed the D9 at (149.6, 145.8)
- removed the D9 at (118.6, 145.8)
- removed the D9 at (87.6, 145.8)
- removed the D9 at (149.6, 79.2)
- removed the D9 at (118.6, 79.2)
- removed the FB1 at (142.2, 142.2)
- removed the FB1 at (111.2, 142.2)
- removed the FB1 at (80.2, 142.2)
- removed the FB1 at (142.2, 75.6)
- removed the FB1 at (111.2, 75.6)
- removed the G*** at (138.9, 134.4)
- removed the G*** at (121.2, 56.9)
- removed the G*** at (108.0, 134.4)
- removed the G*** at (77.0, 134.4)
- removed the G*** at (138.9, 67.8)
- removed the G*** at (108.0, 67.8)
- removed the G*** at (152.1, 123.4)
- removed the G*** at (121.2, 123.4)
- removed the G*** at (90.2, 123.4)
- removed the G*** at (152.1, 56.9)
- removed the H1 at (164.3, 101.9)
- removed the H1 at (133.3, 101.9)
- removed the H1 at (102.4, 101.9)
- removed the H1 at (164.3, 35.3)
- removed the H1 at (133.3, 35.3)
- removed the H2 at (140.0, 101.9)
- removed the H2 at (109.0, 101.9)
- removed the H2 at (78.0, 101.9)
- removed the H2 at (140.0, 35.3)
- removed the H2 at (109.0, 35.3)
- removed the J1 at (139.2, 131.9)
- removed the J1 at (108.2, 131.9)
- removed the J1 at (77.2, 131.9)
- removed the J1 at (139.2, 65.4)
- removed the J1 at (108.2, 65.4)
- removed the J2 at (147.6, 101.0)
- removed the J2 at (116.6, 101.0)
- removed the J2 at (85.6, 101.0)
- removed the J2 at (147.6, 34.4)
- removed the J2 at (116.6, 34.4)
- removed the J3 at (158.2, 160.8)
- removed the J3 at (127.3, 160.8)
- removed the J3 at (96.3, 160.8)
- removed the J3 at (158.2, 94.2)
- removed the J3 at (127.3, 94.2)
- removed the J4 at (165.9, 163.3)
- removed the J4 at (134.9, 163.3)
- removed the J4 at (103.9, 163.3)
- removed the J4 at (165.9, 96.8)
- removed the J4 at (134.9, 96.8)
- removed the J5 at (165.9, 153.2)
- removed the J5 at (134.9, 153.2)
- removed the J5 at (103.9, 153.2)
- removed the J5 at (165.9, 86.6)
- removed the J5 at (134.9, 86.6)
- removed the J6 at (142.2, 162.1)
- removed the J6 at (111.3, 162.1)
- removed the J6 at (80.3, 162.1)
- removed the J6 at (142.2, 95.5)
- removed the J6 at (111.3, 95.5)
- removed the JP2 at (160.3, 158.6)
- removed the JP2 at (129.3, 158.6)
- removed the JP2 at (98.3, 158.6)
- removed the JP2 at (160.3, 92.1)
- removed the JP2 at (129.3, 92.1)
- removed the JP6 at (137.7, 105.7)
- removed the JP6 at (106.7, 105.7)
- removed the JP6 at (75.7, 105.7)
- removed the JP6 at (137.7, 39.1)
- removed the JP6 at (106.7, 39.1)
- removed the JP8 at (157.0, 102.3)
- removed the JP8 at (126.0, 102.3)
- removed the JP8 at (95.0, 102.3)
- removed the JP8 at (157.0, 35.8)
- removed the JP8 at (126.0, 35.8)
- removed the L1 at (142.7, 130.5)
- removed the L1 at (111.7, 130.5)
- removed the L1 at (80.7, 130.5)
- removed the L1 at (142.7, 64.0)
- removed the L1 at (111.7, 64.0)
- removed the Q1 at (149.1, 153.9)
- removed the Q1 at (118.1, 153.9)
- removed the Q1 at (87.1, 153.9)
- removed the Q1 at (149.1, 87.4)
- removed the Q1 at (118.1, 87.4)
- removed the Q2 at (160.8, 109.9)
- removed the Q2 at (129.8, 109.9)
- removed the Q2 at (98.8, 109.9)
- removed the Q2 at (160.8, 43.4)
- removed the Q2 at (129.8, 43.4)
- removed the R1 at (151.3, 121.2)
- removed the R1 at (120.3, 121.2)
- removed the R1 at (89.3, 121.2)
- removed the R1 at (151.3, 54.6)
- removed the R1 at (120.3, 54.6)
- removed the R10 at (141.0, 157.7)
- removed the R10 at (110.0, 157.7)
- removed the R10 at (79.0, 157.7)
- removed the R10 at (141.0, 91.2)
- removed the R10 at (110.0, 91.2)
- removed the R11 at (143.5, 157.7)
- removed the R11 at (112.5, 157.7)
- removed the R11 at (81.5, 157.7)
- removed the R11 at (143.5, 91.2)
- removed the R11 at (112.5, 91.2)
- removed the R12 at (164.8, 128.8)
- removed the R12 at (133.8, 128.8)
- removed the R12 at (102.9, 128.8)
- removed the R12 at (164.8, 62.2)
- removed the R12 at (133.8, 62.2)
- removed the R13 at (164.8, 131.8)
- removed the R13 at (133.9, 131.8)
- removed the R13 at (102.9, 131.8)
- removed the R13 at (164.8, 65.3)
- removed the R13 at (133.9, 65.3)
- removed the R14 at (146.1, 157.7)
- removed the R14 at (115.1, 157.7)
- removed the R14 at (84.1, 157.7)
- removed the R14 at (146.1, 91.2)
- removed the R14 at (115.1, 91.2)
- removed the R15 at (149.1, 149.1)
- removed the R15 at (118.1, 149.1)
- removed the R15 at (87.1, 149.1)
- removed the R15 at (149.1, 82.5)
- removed the R15 at (118.1, 82.5)
- removed the R16 at (153.6, 111.2)
- removed the R16 at (122.6, 111.2)
- removed the R16 at (91.6, 111.2)
- removed the R16 at (153.6, 44.6)
- removed the R16 at (122.6, 44.6)
- removed the R17 at (166.1, 113.7)
- removed the R17 at (135.1, 113.7)
- removed the R17 at (104.1, 113.7)
- removed the R17 at (166.1, 47.1)
- removed the R17 at (135.1, 47.1)
- removed the R18 at (153.4, 121.2)
- removed the R18 at (122.4, 121.2)
- removed the R18 at (91.4, 121.2)
- removed the R18 at (153.4, 54.6)
- removed the R18 at (122.4, 54.6)
- removed the R2 at (149.1, 121.2)
- removed the R2 at (118.1, 121.2)
- removed the R2 at (87.1, 121.2)
- removed the R2 at (149.1, 54.6)
- removed the R2 at (118.1, 54.6)
- removed the R3 at (153.2, 124.4)
- removed the R3 at (122.2, 124.4)
- removed the R3 at (91.2, 124.4)
- removed the R3 at (153.2, 57.8)
- removed the R3 at (122.2, 57.8)
- removed the R4 at (164.8, 134.6)
- removed the R4 at (133.9, 134.6)
- removed the R4 at (102.9, 134.6)
- removed the R4 at (164.8, 68.1)
- removed the R4 at (133.9, 68.1)
- removed the R5 at (153.6, 109.4)
- removed the R5 at (122.6, 109.4)
- removed the R5 at (91.6, 109.4)
- removed the R5 at (153.6, 42.9)
- removed the R5 at (122.6, 42.9)
- removed the R6 at (140.7, 121.2)
- removed the R6 at (109.7, 121.2)
- removed the R6 at (78.7, 121.2)
- removed the R6 at (140.7, 54.6)
- removed the R6 at (109.7, 54.6)
- removed the R7 at (154.4, 143.3)
- removed the R7 at (123.4, 143.3)
- removed the R7 at (92.5, 143.3)
- removed the R7 at (154.4, 76.7)
- removed the R7 at (123.4, 76.7)
- removed the R8 at (138.4, 157.7)
- removed the R8 at (107.4, 157.7)
- removed the R8 at (76.5, 157.7)
- removed the R8 at (138.4, 91.2)
- removed the R8 at (107.4, 91.2)
- removed the R9 at (150.8, 124.4)
- removed the R9 at (119.8, 124.4)
- removed the R9 at (88.8, 124.4)
- removed the R9 at (150.8, 57.8)
- removed the R9 at (119.8, 57.8)
- removed the REF*** at (155.7, 152.1)
- removed the REF*** at (124.7, 152.1)
- removed the REF*** at (93.7, 152.1)
- removed the REF*** at (155.7, 85.6)
- removed the REF*** at (124.7, 85.6)
- removed the S1 at (140.8, 137.6)
- removed the S1 at (109.8, 137.6)
- removed the S1 at (78.8, 137.6)
- removed the S1 at (140.8, 71.0)
- removed the S1 at (109.8, 71.0)
- removed the U1 at (152.1, 133.7)
- removed the U1 at (121.1, 133.7)
- removed the U1 at (90.1, 133.7)
- removed the U1 at (152.1, 67.2)
- removed the U1 at (121.1, 67.2)
- removed the U3 at (141.2, 113.3)
- removed the U3 at (110.2, 113.3)
- removed the U3 at (79.2, 113.3)
- removed the U3 at (141.2, 46.7)
- removed the U3 at (110.2, 46.7)
- removed the U4 at (161.3, 121.2)
- removed the U4 at (130.3, 121.2)
- removed the U4 at (99.3, 121.2)
- removed the U4 at (161.3, 54.6)
- removed the U4 at (130.3, 54.6)
- removed the U5 at (156.0, 152.1)
- removed the U5 at (125.0, 152.1)
- removed the U5 at (94.0, 152.1)
- removed the U5 at (156.0, 85.6)
- removed the U5 at (125.0, 85.6)
- removed the U6 at (158.3, 113.7)
- removed the U6 at (127.3, 113.7)
- removed the U6 at (96.3, 113.7)
- removed the U6 at (158.3, 47.1)
- removed the U6 at (127.3, 47.1)
- removed the Y1 at (149.6, 110.0)
- removed the Y1 at (118.6, 110.0)
- removed the Y1 at (87.6, 110.0)
- removed the Y1 at (149.6, 43.4)
- removed the Y1 at (118.6, 43.4)
- added B1: COIN CELL, SparkX:SparkX-6.8MM_COIN_CELL, F.Cu at (141.1, 146.9)
- added B1: COIN CELL, SparkX:SparkX-6.8MM_COIN_CELL, F.Cu at (110.1, 146.9)
- added B1: COIN CELL, SparkX:SparkX-6.8MM_COIN_CELL, F.Cu at (79.2, 146.9)
- added B1: COIN CELL, SparkX:SparkX-6.8MM_COIN_CELL, F.Cu at (141.1, 80.4)
- added B1: COIN CELL, SparkX:SparkX-6.8MM_COIN_CELL, F.Cu at (110.1, 80.4)
- added C1: 10pF, Capacitors_SMD:C_0603, F.Cu at (127.4, 119.7)
- added C1: 10pF, Capacitors_SMD:C_0603, F.Cu at (96.4, 119.7)
- added C1: 10pF, Capacitors_SMD:C_0603, F.Cu at (65.4, 119.7)
- added C1: 10pF, Capacitors_SMD:C_0603, F.Cu at (127.4, 53.1)
- added C1: 10pF, Capacitors_SMD:C_0603, F.Cu at (96.4, 53.1)
- added C10: 0.1uF, Capacitors_SMD:C_0603, F.Cu at (115.8, 128.3)
- added C10: 0.1uF, Capacitors_SMD:C_0603, F.Cu at (84.8, 128.3)
- added C10: 0.1uF, Capacitors_SMD:C_0603, F.Cu at (53.8, 128.3)
- added C10: 0.1uF, Capacitors_SMD:C_0603, F.Cu at (115.8, 61.7)
- added C10: 0.1uF, Capacitors_SMD:C_0603, F.Cu at (84.8, 61.7)
- added C11: 0.1uF, Capacitors_SMD:C_0603, F.Cu at (134.6, 128.3)
- added C11: 0.1uF, Capacitors_SMD:C_0603, F.Cu at (103.6, 128.3)
- added C11: 0.1uF, Capacitors_SMD:C_0603, F.Cu at (72.6, 128.3)
- added C11: 0.1uF, Capacitors_SMD:C_0603, F.Cu at (134.6, 61.7)
- added C11: 0.1uF, Capacitors_SMD:C_0603, F.Cu at (103.6, 61.7)
- added C12: 1.0uF, Capacitors_SMD:C_0603, F.Cu at (120.7, 131.3)
- added C12: 1.0uF, Capacitors_SMD:C_0603, F.Cu at (89.7, 131.3)
- added C12: 1.0uF, Capacitors_SMD:C_0603, F.Cu at (58.7, 131.3)
- added C12: 1.0uF, Capacitors_SMD:C_0603, F.Cu at (120.7, 64.8)
- added C12: 1.0uF, Capacitors_SMD:C_0603, F.Cu at (89.7, 64.8)
- added C13: 0.1uF, Capacitors_SMD:C_0603, F.Cu at (121.8, 149.3)
- added C13: 0.1uF, Capacitors_SMD:C_0603, F.Cu at (90.8, 149.3)
- added C13: 0.1uF, Capacitors_SMD:C_0603, F.Cu at (59.8, 149.3)
- added C13: 0.1uF, Capacitors_SMD:C_0603, F.Cu at (121.8, 82.7)
- added C13: 0.1uF, Capacitors_SMD:C_0603, F.Cu at (90.8, 82.7)
- added C14: 1.0uF, Capacitors_SMD:C_0603, F.Cu at (124.0, 149.3)
- added C14: 1.0uF, Capacitors_SMD:C_0603, F.Cu at (93.0, 149.3)
- added C14: 1.0uF, Capacitors_SMD:C_0603, F.Cu at (62.0, 149.3)
- added C14: 1.0uF, Capacitors_SMD:C_0603, F.Cu at (124.0, 82.7)
- added C14: 1.0uF, Capacitors_SMD:C_0603, F.Cu at (93.0, 82.7)
- added C15: 4.7uF, Capacitors_SMD:C_0603, F.Cu at (141.2, 120.8)
- added C15: 4.7uF, Capacitors_SMD:C_0603, F.Cu at (110.2, 120.8)
- added C15: 4.7uF, Capacitors_SMD:C_0603, F.Cu at (79.2, 120.8)
- added C15: 4.7uF, Capacitors_SMD:C_0603, F.Cu at (141.2, 54.2)
- added C15: 4.7uF, Capacitors_SMD:C_0603, F.Cu at (110.2, 54.2)
- added C2: 10pF, Capacitors_SMD:C_0603, F.Cu at (127.4, 114.6)
- added C2: 10pF, Capacitors_SMD:C_0603, F.Cu at (96.4, 114.6)
- added C2: 10pF, Capacitors_SMD:C_0603, F.Cu at (65.4, 114.6)
- added C2: 10pF, Capacitors_SMD:C_0603, F.Cu at (127.4, 48.0)
- added C2: 10pF, Capacitors_SMD:C_0603, F.Cu at (96.4, 48.0)
- added C3: 10nF, Capacitors_SMD:C_0603, F.Cu at (125.0, 121.8)
- added C3: 10nF, Capacitors_SMD:C_0603, F.Cu at (94.0, 121.8)
- added C3: 10nF, Capacitors_SMD:C_0603, F.Cu at (63.0, 121.8)
- added C3: 10nF, Capacitors_SMD:C_0603, F.Cu at (125.0, 55.2)
- added C3: 10nF, Capacitors_SMD:C_0603, F.Cu at (94.0, 55.2)
- added C4: 0.1uF, Capacitors_SMD:C_0603, F.Cu at (124.8, 131.5)
- added C4: 0.1uF, Capacitors_SMD:C_0603, F.Cu at (93.8, 131.5)
- added C4: 0.1uF, Capacitors_SMD:C_0603, F.Cu at (62.8, 131.5)
- added C4: 0.1uF, Capacitors_SMD:C_0603, F.Cu at (124.8, 64.9)
- added C4: 0.1uF, Capacitors_SMD:C_0603, F.Cu at (93.8, 64.9)
- added C5: 4.7uF, Capacitors_SMD:C_0603, F.Cu at (139.0, 120.8)
- added C5: 4.7uF, Capacitors_SMD:C_0603, F.Cu at (108.0, 120.8)
- added C5: 4.7uF, Capacitors_SMD:C_0603, F.Cu at (77.0, 120.8)
- added C5: 4.7uF, Capacitors_SMD:C_0603, F.Cu at (139.0, 54.2)
- added C5: 4.7uF, Capacitors_SMD:C_0603, F.Cu at (108.0, 54.2)
- added C6: 1.0uF, Capacitors_SMD:C_0603, F.Cu at (143.0, 128.3)
- added C6: 1.0uF, Capacitors_SMD:C_0603, F.Cu at (112.0, 128.3)
- added C6: 1.0uF, Capacitors_SMD:C_0603, F.Cu at (81.0, 128.3)
- added C6: 1.0uF, Capacitors_SMD:C_0603, F.Cu at (143.0, 61.7)
- added C6: 1.0uF, Capacitors_SMD:C_0603, F.Cu at (112.0, 61.7)
- added C7: 2.2uF, Capacitors_SMD:C_0603, F.Cu at (140.5, 125.2)
- added C7: 2.2uF, Capacitors_SMD:C_0603, F.Cu at (109.5, 125.2)
- added C7: 2.2uF, Capacitors_SMD:C_0603, F.Cu at (78.5, 125.2)
- added C7: 2.2uF, Capacitors_SMD:C_0603, F.Cu at (140.5, 58.7)
- added C7: 2.2uF, Capacitors_SMD:C_0603, F.Cu at (109.5, 58.7)
- added C8: 1.0uF, Capacitors_SMD:C_0603, F.Cu at (127.0, 150.4)
- added C8: 1.0uF, Capacitors_SMD:C_0603, F.Cu at (96.0, 150.4)
- added C8: 1.0uF, Capacitors_SMD:C_0603, F.Cu at (65.0, 150.4)
- added C8: 1.0uF, Capacitors_SMD:C_0603, F.Cu at (127.0, 83.8)
- added C8: 1.0uF, Capacitors_SMD:C_0603, F.Cu at (96.0, 83.8)
- added C9: 0.1uF, Capacitors_SMD:C_0603, F.Cu at (122.9, 128.3)
- added C9: 0.1uF, Capacitors_SMD:C_0603, F.Cu at (91.9, 128.3)
- added C9: 0.1uF, Capacitors_SMD:C_0603, F.Cu at (61.0, 128.3)
- added C9: 0.1uF, Capacitors_SMD:C_0603, F.Cu at (122.9, 61.7)
- added C9: 0.1uF, Capacitors_SMD:C_0603, F.Cu at (91.9, 61.7)
- added D1: Blue, LEDs:LED_0603, F.Cu at (134.2, 131.5)
- added D1: Blue, LEDs:LED_0603, F.Cu at (103.2, 131.5)
- added D1: Blue, LEDs:LED_0603, F.Cu at (72.2, 131.5)
- added D1: Blue, LEDs:LED_0603, F.Cu at (134.2, 64.9)
- added D1: Blue, LEDs:LED_0603, F.Cu at (103.2, 64.9)
- added D10: BAT20J, DiscreteSemi:SparkFun-DiscreteSemi-SOD-323, F.Cu at (141.2, 117.0)
- added D10: BAT20J, DiscreteSemi:SparkFun-DiscreteSemi-SOD-323, F.Cu at (110.2, 117.0)
- added D10: BAT20J, DiscreteSemi:SparkFun-DiscreteSemi-SOD-323, F.Cu at (79.2, 117.0)
- added D10: BAT20J, DiscreteSemi:SparkFun-DiscreteSemi-SOD-323, F.Cu at (141.2, 50.5)
- added D10: BAT20J, DiscreteSemi:SparkFun-DiscreteSemi-SOD-323, F.Cu at (110.2, 50.5)
- added D11: Yellow, LEDs:LED_0603, F.Cu at (136.4, 125.5)
- added D11: Yellow, LEDs:LED_0603, F.Cu at (105.4, 125.5)
- added D11: Yellow, LEDs:LED_0603, F.Cu at (74.4, 125.5)
- added D11: Yellow, LEDs:LED_0603, F.Cu at (136.4, 58.9)
- added D11: Yellow, LEDs:LED_0603, F.Cu at (105.4, 58.9)
- added D12: Red, LEDs:LED_0603, F.Cu at (132.3, 125.5)
- added D12: Red, LEDs:LED_0603, F.Cu at (101.3, 125.5)
- added D12: Red, LEDs:LED_0603, F.Cu at (70.4, 125.5)
- added D12: Red, LEDs:LED_0603, F.Cu at (132.3, 58.9)
- added D12: Red, LEDs:LED_0603, F.Cu at (101.3, 58.9)
- added D2: 0.5A/40V/420mV, DiscreteSemi:SparkFun-DiscreteSemi-SOD-323, F.Cu at (139.2, 140.7)
- added D2: 0.5A/40V/420mV, DiscreteSemi:SparkFun-DiscreteSemi-SOD-323, F.Cu at (108.2, 140.7)
- added D2: 0.5A/40V/420mV, DiscreteSemi:SparkFun-DiscreteSemi-SOD-323, F.Cu at (77.2, 140.7)
- added D2: 0.5A/40V/420mV, DiscreteSemi:SparkFun-DiscreteSemi-SOD-323, F.Cu at (139.2, 74.2)
- added D2: 0.5A/40V/420mV, DiscreteSemi:SparkFun-DiscreteSemi-SOD-323, F.Cu at (108.2, 74.2)
- added D3: Yellow, LEDs:LED_0603, F.Cu at (128.8, 125.5)
- added D3: Yellow, LEDs:LED_0603, F.Cu at (97.8, 125.5)
- added D3: Yellow, LEDs:LED_0603, F.Cu at (66.8, 125.5)
- added D3: Yellow, LEDs:LED_0603, F.Cu at (128.8, 58.9)
- added D3: Yellow, LEDs:LED_0603, F.Cu at (97.8, 58.9)
- added D4: GREEN, LEDs:LED_0603, F.Cu at (124.9, 125.5)
- added D4: GREEN, LEDs:LED_0603, F.Cu at (93.9, 125.5)
- added D4: GREEN, LEDs:LED_0603, F.Cu at (63.0, 125.5)
- added D4: GREEN, LEDs:LED_0603, F.Cu at (124.9, 58.9)
- added D4: GREEN, LEDs:LED_0603, F.Cu at (93.9, 58.9)
- added D5: Blue, LEDs:LED_0603, F.Cu at (115.8, 162.1)
- added D5: Blue, LEDs:LED_0603, F.Cu at (84.8, 162.1)
- added D5: Blue, LEDs:LED_0603, F.Cu at (53.8, 162.1)
- added D5: Blue, LEDs:LED_0603, F.Cu at (115.8, 95.5)
- added D5: Blue, LEDs:LED_0603, F.Cu at (84.8, 95.5)
- added D6: Blue, LEDs:LED_0603, F.Cu at (118.4, 162.1)
- added D6: Blue, LEDs:LED_0603, F.Cu at (87.4, 162.1)
- added D6: Blue, LEDs:LED_0603, F.Cu at (56.4, 162.1)
- added D6: Blue, LEDs:LED_0603, F.Cu at (118.4, 95.5)
- added D6: Blue, LEDs:LED_0603, F.Cu at (87.4, 95.5)
- added D7: Blue, LEDs:LED_0603, F.Cu at (120.9, 162.1)
- added D7: Blue, LEDs:LED_0603, F.Cu at (89.9, 162.1)
- added D7: Blue, LEDs:LED_0603, F.Cu at (58.9, 162.1)
- added D7: Blue, LEDs:LED_0603, F.Cu at (120.9, 95.5)
- added D7: Blue, LEDs:LED_0603, F.Cu at (89.9, 95.5)
- added D8: Blue, LEDs:LED_0603, F.Cu at (123.4, 162.0)
- added D8: Blue, LEDs:LED_0603, F.Cu at (92.5, 162.0)
- added D8: Blue, LEDs:LED_0603, F.Cu at (61.5, 162.0)
- added D8: Blue, LEDs:LED_0603, F.Cu at (123.4, 95.5)
- added D8: Blue, LEDs:LED_0603, F.Cu at (92.5, 95.5)
- added D9: Blue, LEDs:LED_0603, F.Cu at (127.0, 152.9)
- added D9: Blue, LEDs:LED_0603, F.Cu at (96.0, 152.9)
- added D9: Blue, LEDs:LED_0603, F.Cu at (65.0, 152.9)
- added D9: Blue, LEDs:LED_0603, F.Cu at (127.0, 86.4)
- added D9: Blue, LEDs:LED_0603, F.Cu at (96.0, 86.4)
- added FB1: 600Ohm/100MHz, Inductors_SMD:L_0603, F.Cu at (119.6, 149.3)
- added FB1: 600Ohm/100MHz, Inductors_SMD:L_0603, F.Cu at (88.6, 149.3)
- added FB1: 600Ohm/100MHz, Inductors_SMD:L_0603, F.Cu at (57.6, 149.3)
- added FB1: 600Ohm/100MHz, Inductors_SMD:L_0603, F.Cu at (119.6, 82.7)
- added FB1: 600Ohm/100MHz, Inductors_SMD:L_0603, F.Cu at (88.6, 82.7)
- added G***: LOGO, Custom_Silk:SparkX_Logo, B.Cu at (116.3, 141.5)
- added G***: LOGO, Custom_Silk:worldmap_silk, B.Cu at (98.6, 64.0)
- added G***: LOGO, Custom_Silk:SparkX_Logo, B.Cu at (85.3, 141.5)
- added G***: LOGO, Custom_Silk:SparkX_Logo, B.Cu at (54.4, 141.5)
- added G***: LOGO, Custom_Silk:SparkX_Logo, B.Cu at (116.3, 74.9)
- added G***: LOGO, Custom_Silk:SparkX_Logo, B.Cu at (85.3, 74.9)
- added G***: LOGO, Custom_Silk:worldmap_silk, B.Cu at (129.5, 130.6)
- added G***: LOGO, Custom_Silk:worldmap_silk, B.Cu at (98.6, 130.6)
- added G***: LOGO, Custom_Silk:worldmap_silk, B.Cu at (67.6, 130.6)
- added G***: LOGO, Custom_Silk:worldmap_silk, B.Cu at (129.5, 64.0)
- added H1: STAND-OFF, Hardware:STAND-OFF, F.Cu at (141.7, 109.0)
- added H1: STAND-OFF, Hardware:STAND-OFF, F.Cu at (110.7, 109.0)
- added H1: STAND-OFF, Hardware:STAND-OFF, F.Cu at (79.8, 109.0)
- added H1: STAND-OFF, Hardware:STAND-OFF, F.Cu at (141.7, 42.4)
- added H1: STAND-OFF, Hardware:STAND-OFF, F.Cu at (110.7, 42.4)
- added H2: STAND-OFF, Hardware:STAND-OFF, F.Cu at (117.3, 109.0)
- added H2: STAND-OFF, Hardware:STAND-OFF, F.Cu at (86.4, 109.0)
- added H2: STAND-OFF, Hardware:STAND-OFF, F.Cu at (55.4, 109.0)
- added H2: STAND-OFF, Hardware:STAND-OFF, F.Cu at (117.3, 42.4)
- added H2: STAND-OFF, Hardware:STAND-OFF, F.Cu at (86.4, 42.4)
- added J1: U.FL, SparkX:SparkX-U.FL, F.Cu at (116.6, 139.0)
- added J1: U.FL, SparkX:SparkX-U.FL, F.Cu at (85.6, 139.0)
- added J1: U.FL, SparkX:SparkX-U.FL, F.Cu at (54.6, 139.0)
- added J1: U.FL, SparkX:SparkX-U.FL, F.Cu at (116.6, 72.5)
- added J1: U.FL, SparkX:SparkX-U.FL, F.Cu at (85.6, 72.5)
- added J2: microB, Connectors:USB-B-MICRO-SMD, F.Cu at (125.0, 108.1)
- added J2: microB, Connectors:USB-B-MICRO-SMD, F.Cu at (94.0, 108.1)
- added J2: microB, Connectors:USB-B-MICRO-SMD, F.Cu at (63.0, 108.1)
- added J2: microB, Connectors:USB-B-MICRO-SMD, F.Cu at (125.0, 41.5)
- added J2: microB, Connectors:USB-B-MICRO-SMD, F.Cu at (94.0, 41.5)
- added J3: AVR_SPI_PROG_3X2PTH, Connectors:2X3, F.Cu at (135.6, 167.9)
- added J3: AVR_SPI_PROG_3X2PTH, Connectors:2X3, F.Cu at (104.6, 167.9)
- added J3: AVR_SPI_PROG_3X2PTH, Connectors:2X3, F.Cu at (73.7, 167.9)
- added J3: AVR_SPI_PROG_3X2PTH, Connectors:2X3, F.Cu at (135.6, 101.3)
- added J3: AVR_SPI_PROG_3X2PTH, Connectors:2X3, F.Cu at (104.6, 101.3)
- added J4: CONN_04, Connectors:1X04, F.Cu at (143.3, 170.4)
- added J4: CONN_04, Connectors:1X04, F.Cu at (112.3, 170.4)
- added J4: CONN_04, Connectors:1X04, F.Cu at (81.3, 170.4)
- added J4: CONN_04, Connectors:1X04, F.Cu at (143.3, 103.9)
- added J4: CONN_04, Connectors:1X04, F.Cu at (112.3, 103.9)
- added J5: CONN_04, Connectors:1X04, F.Cu at (143.3, 160.3)
- added J5: CONN_04, Connectors:1X04, F.Cu at (112.3, 160.3)
- added J5: CONN_04, Connectors:1X04, F.Cu at (81.3, 160.3)
- added J5: CONN_04, Connectors:1X04, F.Cu at (143.3, 93.7)
- added J5: CONN_04, Connectors:1X04, F.Cu at (112.3, 93.7)
- added J6: CONN_04X2, Connectors:2X4, F.Cu at (119.6, 169.2)
- added J6: CONN_04X2, Connectors:2X4, F.Cu at (88.6, 169.2)
- added J6: CONN_04X2, Connectors:2X4, F.Cu at (57.7, 169.2)
- added J6: CONN_04X2, Connectors:2X4, F.Cu at (119.6, 102.6)
- added J6: CONN_04X2, Connectors:2X4, F.Cu at (88.6, 102.6)
- added JP2: FIDUCIALUFIDUCIAL, Aesthetics:FIDUCIAL-MICRO, F.Cu at (137.7, 165.7)
- added JP2: FIDUCIALUFIDUCIAL, Aesthetics:FIDUCIAL-MICRO, F.Cu at (106.7, 165.7)
- added JP2: FIDUCIALUFIDUCIAL, Aesthetics:FIDUCIAL-MICRO, F.Cu at (75.7, 165.7)
- added JP2: FIDUCIALUFIDUCIAL, Aesthetics:FIDUCIAL-MICRO, F.Cu at (137.7, 99.2)
- added JP2: FIDUCIALUFIDUCIAL, Aesthetics:FIDUCIAL-MICRO, F.Cu at (106.7, 99.2)
- added JP6: FIDUCIALUFIDUCIAL, Aesthetics:FIDUCIAL-MICRO, F.Cu at (115.1, 112.8)
- added JP6: FIDUCIALUFIDUCIAL, Aesthetics:FIDUCIAL-MICRO, F.Cu at (84.1, 112.8)
- added JP6: FIDUCIALUFIDUCIAL, Aesthetics:FIDUCIAL-MICRO, F.Cu at (53.1, 112.8)
- added JP6: FIDUCIALUFIDUCIAL, Aesthetics:FIDUCIAL-MICRO, F.Cu at (115.1, 46.2)
- added JP6: FIDUCIALUFIDUCIAL, Aesthetics:FIDUCIAL-MICRO, F.Cu at (84.1, 46.2)
- added JP8: LiPo, Connectors:JST-2-SMD, F.Cu at (134.4, 109.4)
- added JP8: LiPo, Connectors:JST-2-SMD, F.Cu at (103.4, 109.4)
- added JP8: LiPo, Connectors:JST-2-SMD, F.Cu at (72.4, 109.4)
- added JP8: LiPo, Connectors:JST-2-SMD, F.Cu at (134.4, 42.9)
- added JP8: LiPo, Connectors:JST-2-SMD, F.Cu at (103.4, 42.9)
- added L1: 33nH/~5%/500mA, Inductors_SMD:L_0603, F.Cu at (120.1, 137.6)
- added L1: 33nH/~5%/500mA, Inductors_SMD:L_0603, F.Cu at (89.1, 137.6)
- added L1: 33nH/~5%/500mA, Inductors_SMD:L_0603, F.Cu at (58.1, 137.6)
- added L1: 33nH/~5%/500mA, Inductors_SMD:L_0603, F.Cu at (120.1, 71.1)
- added L1: 33nH/~5%/500mA, Inductors_SMD:L_0603, F.Cu at (89.1, 71.1)
- added Q1: 8/16/20MHz, Clocks:RESONATOR-SMD-3.2X1.3, F.Cu at (126.5, 161.0)
- added Q1: 8/16/20MHz, Clocks:RESONATOR-SMD-3.2X1.3, F.Cu at (95.5, 161.0)
- added Q1: 8/16/20MHz, Clocks:RESONATOR-SMD-3.2X1.3, F.Cu at (64.5, 161.0)
- added Q1: 8/16/20MHz, Clocks:RESONATOR-SMD-3.2X1.3, F.Cu at (126.5, 94.5)
- added Q1: 8/16/20MHz, Clocks:RESONATOR-SMD-3.2X1.3, F.Cu at (95.5, 94.5)
- added Q2: 2.5A/30V, DiscreteSemi:SparkFun-DiscreteSemi-SOT23-3, F.Cu at (138.2, 117.0)
- added Q2: 2.5A/30V, DiscreteSemi:SparkFun-DiscreteSemi-SOT23-3, F.Cu at (107.2, 117.0)
- added Q2: 2.5A/30V, DiscreteSemi:SparkFun-DiscreteSemi-SOT23-3, F.Cu at (76.2, 117.0)
- added Q2: 2.5A/30V, DiscreteSemi:SparkFun-DiscreteSemi-SOT23-3, F.Cu at (138.2, 50.5)
- added Q2: 2.5A/30V, DiscreteSemi:SparkFun-DiscreteSemi-SOT23-3, F.Cu at (107.2, 50.5)
- added R1: 1k, Resistors_SMD:R_0603, F.Cu at (128.7, 128.3)
- added R1: 1k, Resistors_SMD:R_0603, F.Cu at (97.7, 128.3)
- added R1: 1k, Resistors_SMD:R_0603, F.Cu at (66.7, 128.3)
- added R1: 1k, Resistors_SMD:R_0603, F.Cu at (128.7, 61.7)
- added R1: 1k, Resistors_SMD:R_0603, F.Cu at (97.7, 61.7)
- added R10: 470, Resistors_SMD:R_0603, F.Cu at (118.4, 164.9)
- added R10: 470, Resistors_SMD:R_0603, F.Cu at (87.4, 164.9)
- added R10: 470, Resistors_SMD:R_0603, F.Cu at (56.4, 164.9)
- added R10: 470, Resistors_SMD:R_0603, F.Cu at (118.4, 98.3)
- added R10: 470, Resistors_SMD:R_0603, F.Cu at (87.4, 98.3)
- added R11: 470, Resistors_SMD:R_0603, F.Cu at (120.9, 164.8)
- added R11: 470, Resistors_SMD:R_0603, F.Cu at (89.9, 164.8)
- added R11: 470, Resistors_SMD:R_0603, F.Cu at (58.9, 164.8)
- added R11: 470, Resistors_SMD:R_0603, F.Cu at (120.9, 98.3)
- added R11: 470, Resistors_SMD:R_0603, F.Cu at (89.9, 98.3)
- added R12: 4.7k, Resistors_SMD:R_0603, F.Cu at (142.2, 135.9)
- added R12: 4.7k, Resistors_SMD:R_0603, F.Cu at (111.2, 135.9)
- added R12: 4.7k, Resistors_SMD:R_0603, F.Cu at (80.3, 135.9)
- added R12: 4.7k, Resistors_SMD:R_0603, F.Cu at (142.2, 69.3)
- added R12: 4.7k, Resistors_SMD:R_0603, F.Cu at (111.2, 69.3)
- added R13: 4.7k, Resistors_SMD:R_0603, F.Cu at (142.2, 138.9)
- added R13: 4.7k, Resistors_SMD:R_0603, F.Cu at (111.3, 138.9)
- added R13: 4.7k, Resistors_SMD:R_0603, F.Cu at (80.3, 138.9)
- added R13: 4.7k, Resistors_SMD:R_0603, F.Cu at (142.2, 72.4)
- added R13: 4.7k, Resistors_SMD:R_0603, F.Cu at (111.3, 72.4)
- added R14: 470, Resistors_SMD:R_0603, F.Cu at (123.4, 164.8)
- added R14: 470, Resistors_SMD:R_0603, F.Cu at (92.5, 164.8)
- added R14: 470, Resistors_SMD:R_0603, F.Cu at (61.5, 164.8)
- added R14: 470, Resistors_SMD:R_0603, F.Cu at (123.4, 98.3)
- added R14: 470, Resistors_SMD:R_0603, F.Cu at (92.5, 98.3)
- added R15: 470, Resistors_SMD:R_0603, F.Cu at (126.5, 156.2)
- added R15: 470, Resistors_SMD:R_0603, F.Cu at (95.5, 156.2)
- added R15: 470, Resistors_SMD:R_0603, F.Cu at (64.5, 156.2)
- added R15: 470, Resistors_SMD:R_0603, F.Cu at (126.5, 89.7)
- added R15: 470, Resistors_SMD:R_0603, F.Cu at (95.5, 89.7)
- added R16: 2.0k, Resistors_SMD:R_0603, F.Cu at (131.0, 118.3)
- added R16: 2.0k, Resistors_SMD:R_0603, F.Cu at (100.0, 118.3)
- added R16: 2.0k, Resistors_SMD:R_0603, F.Cu at (69.0, 118.3)
- added R16: 2.0k, Resistors_SMD:R_0603, F.Cu at (131.0, 51.7)
- added R16: 2.0k, Resistors_SMD:R_0603, F.Cu at (100.0, 51.7)
- added R17: 1k, Resistors_SMD:R_0603, F.Cu at (143.5, 120.8)
- added R17: 1k, Resistors_SMD:R_0603, F.Cu at (112.5, 120.8)
- added R17: 1k, Resistors_SMD:R_0603, F.Cu at (81.5, 120.8)
- added R17: 1k, Resistors_SMD:R_0603, F.Cu at (143.5, 54.2)
- added R17: 1k, Resistors_SMD:R_0603, F.Cu at (112.5, 54.2)
- added R18: 1k, Resistors_SMD:R_0603, F.Cu at (130.8, 128.3)
- added R18: 1k, Resistors_SMD:R_0603, F.Cu at (99.8, 128.3)
- added R18: 1k, Resistors_SMD:R_0603, F.Cu at (68.8, 128.3)
- added R18: 1k, Resistors_SMD:R_0603, F.Cu at (130.8, 61.7)
- added R18: 1k, Resistors_SMD:R_0603, F.Cu at (99.8, 61.7)
- added R2: 470, Resistors_SMD:R_0603, F.Cu at (126.5, 128.3)
- added R2: 470, Resistors_SMD:R_0603, F.Cu at (95.5, 128.3)
- added R2: 470, Resistors_SMD:R_0603, F.Cu at (64.5, 128.3)
- added R2: 470, Resistors_SMD:R_0603, F.Cu at (126.5, 61.7)
- added R2: 470, Resistors_SMD:R_0603, F.Cu at (95.5, 61.7)
- added R3: 470, Resistors_SMD:R_0603, F.Cu at (130.6, 131.5)
- added R3: 470, Resistors_SMD:R_0603, F.Cu at (99.6, 131.5)
- added R3: 470, Resistors_SMD:R_0603, F.Cu at (68.6, 131.5)
- added R3: 470, Resistors_SMD:R_0603, F.Cu at (130.6, 64.9)
- added R3: 470, Resistors_SMD:R_0603, F.Cu at (99.6, 64.9)
- added R4: 1k, Resistors_SMD:R_0603, F.Cu at (142.2, 141.7)
- added R4: 1k, Resistors_SMD:R_0603, F.Cu at (111.3, 141.7)
- added R4: 1k, Resistors_SMD:R_0603, F.Cu at (80.3, 141.7)
- added R4: 1k, Resistors_SMD:R_0603, F.Cu at (142.2, 75.2)
- added R4: 1k, Resistors_SMD:R_0603, F.Cu at (111.3, 75.2)
- added R5: 10k, Resistors_SMD:R_0603, F.Cu at (131.0, 116.5)
- added R5: 10k, Resistors_SMD:R_0603, F.Cu at (100.0, 116.5)
- added R5: 10k, Resistors_SMD:R_0603, F.Cu at (69.0, 116.5)
- added R5: 10k, Resistors_SMD:R_0603, F.Cu at (131.0, 50.0)
- added R5: 10k, Resistors_SMD:R_0603, F.Cu at (100.0, 50.0)
- added R6: 10k, Resistors_SMD:R_0603, F.Cu at (118.1, 128.3)
- added R6: 10k, Resistors_SMD:R_0603, F.Cu at (87.1, 128.3)
- added R6: 10k, Resistors_SMD:R_0603, F.Cu at (56.1, 128.3)
- added R6: 10k, Resistors_SMD:R_0603, F.Cu at (118.1, 61.7)
- added R6: 10k, Resistors_SMD:R_0603, F.Cu at (87.1, 61.7)
- added R7: 10k, Resistors_SMD:R_0603, F.Cu at (131.8, 150.4)
- added R7: 10k, Resistors_SMD:R_0603, F.Cu at (100.8, 150.4)
- added R7: 10k, Resistors_SMD:R_0603, F.Cu at (69.8, 150.4)
- added R7: 10k, Resistors_SMD:R_0603, F.Cu at (131.8, 83.8)
- added R7: 10k, Resistors_SMD:R_0603, F.Cu at (100.8, 83.8)
- added R8: 470, Resistors_SMD:R_0603, F.Cu at (115.8, 164.8)
- added R8: 470, Resistors_SMD:R_0603, F.Cu at (84.8, 164.8)
- added R8: 470, Resistors_SMD:R_0603, F.Cu at (53.8, 164.8)
- added R8: 470, Resistors_SMD:R_0603, F.Cu at (115.8, 98.3)
- added R8: 470, Resistors_SMD:R_0603, F.Cu at (84.8, 98.3)
- added R9: 10k, Resistors_SMD:R_0603, F.Cu at (128.2, 131.5)
- added R9: 10k, Resistors_SMD:R_0603, F.Cu at (97.2, 131.5)
- added R9: 10k, Resistors_SMD:R_0603, F.Cu at (66.2, 131.5)
- added R9: 10k, Resistors_SMD:R_0603, F.Cu at (128.2, 64.9)
- added R9: 10k, Resistors_SMD:R_0603, F.Cu at (97.2, 64.9)
- added REF***: OSHW-Symbol_6.7x6mm_SilkScreen, Symbols:OSHW-Symbol_6.7x6mm_SilkScreen, B.Cu at (133.1, 159.3)
- added REF***: OSHW-Symbol_6.7x6mm_SilkScreen, Symbols:OSHW-Symbol_6.7x6mm_SilkScreen, B.Cu at (102.1, 159.3)
- added REF***: OSHW-Symbol_6.7x6mm_SilkScreen, Symbols:OSHW-Symbol_6.7x6mm_SilkScreen, B.Cu at (71.1, 159.3)
- added REF***: OSHW-Symbol_6.7x6mm_SilkScreen, Symbols:OSHW-Symbol_6.7x6mm_SilkScreen, B.Cu at (133.1, 92.7)
- added REF***: OSHW-Symbol_6.7x6mm_SilkScreen, Symbols:OSHW-Symbol_6.7x6mm_SilkScreen, B.Cu at (102.1, 92.7)
- added S1: Reset, Switches:TACTILE_SWITCH_SMD_5.2MM, F.Cu at (118.2, 144.7)
- added S1: Reset, Switches:TACTILE_SWITCH_SMD_5.2MM, F.Cu at (87.2, 144.7)
- added S1: Reset, Switches:TACTILE_SWITCH_SMD_5.2MM, F.Cu at (56.2, 144.7)
- added S1: Reset, Switches:TACTILE_SWITCH_SMD_5.2MM, F.Cu at (118.2, 78.1)
- added S1: Reset, Switches:TACTILE_SWITCH_SMD_5.2MM, F.Cu at (87.2, 78.1)
- added U1: TITAN X1 GPS, SparkX:SparkX-TITAN_X1_GPS, F.Cu at (129.5, 140.8)
- added U1: TITAN X1 GPS, SparkX:SparkX-TITAN_X1_GPS, F.Cu at (98.5, 140.8)
- added U1: TITAN X1 GPS, SparkX:SparkX-TITAN_X1_GPS, F.Cu at (67.5, 140.8)
- added U1: TITAN X1 GPS, SparkX:SparkX-TITAN_X1_GPS, F.Cu at (129.5, 74.3)
- added U1: TITAN X1 GPS, SparkX:SparkX-TITAN_X1_GPS, F.Cu at (98.5, 74.3)
- added U3: CH340G, IC:SO16, F.Cu at (118.6, 120.4)
- added U3: CH340G, IC:SO16, F.Cu at (87.6, 120.4)
- added U3: CH340G, IC:SO16, F.Cu at (56.6, 120.4)
- added U3: CH340G, IC:SO16, F.Cu at (118.6, 53.8)
- added U3: CH340G, IC:SO16, F.Cu at (87.6, 53.8)
- added U4: AP2112K-3.3V, IC:SOT23-5, F.Cu at (138.7, 128.3)
- added U4: AP2112K-3.3V, IC:SOT23-5, F.Cu at (107.7, 128.3)
- added U4: AP2112K-3.3V, IC:SOT23-5, F.Cu at (76.7, 128.3)
- added U4: AP2112K-3.3V, IC:SOT23-5, F.Cu at (138.7, 61.7)
- added U4: AP2112K-3.3V, IC:SOT23-5, F.Cu at (107.7, 61.7)
- added U5: ATMEGA328, IC:TQFP32-08, F.Cu at (133.3, 159.3)
- added U5: ATMEGA328, IC:TQFP32-08, F.Cu at (102.4, 159.3)
- added U5: ATMEGA328, IC:TQFP32-08, F.Cu at (71.4, 159.3)
- added U5: ATMEGA328, IC:TQFP32-08, F.Cu at (133.3, 92.7)
- added U5: ATMEGA328, IC:TQFP32-08, F.Cu at (102.4, 92.7)
- added U6: MCP73831, IC:SOT23-5, F.Cu at (135.7, 120.8)
- added U6: MCP73831, IC:SOT23-5, F.Cu at (104.7, 120.8)
- added U6: MCP73831, IC:SOT23-5, F.Cu at (73.7, 120.8)
- added U6: MCP73831, IC:SOT23-5, F.Cu at (135.7, 54.2)
- added U6: MCP73831, IC:SOT23-5, F.Cu at (104.7, 54.2)
- added Y1: 12MHz, Clocks:CRYSTAL-SMD-3.2X2.5MM, F.Cu at (127.0, 117.1)
- added Y1: 12MHz, Clocks:CRYSTAL-SMD-3.2X2.5MM, F.Cu at (96.0, 117.1)
- added Y1: 12MHz, Clocks:CRYSTAL-SMD-3.2X2.5MM, F.Cu at (65.0, 117.1)
- added Y1: 12MHz, Clocks:CRYSTAL-SMD-3.2X2.5MM, F.Cu at (127.0, 50.5)
- added Y1: 12MHz, Clocks:CRYSTAL-SMD-3.2X2.5MM, F.Cu at (96.0, 50.5)
- moved B1 23.7 mm to (79.2, 80.4)
- moved C14 23.7 mm to (62.0, 82.7)
- moved C6 23.7 mm to (81.0, 61.7)
- moved D11 23.7 mm to (74.4, 58.9)
- moved D2 23.7 mm to (77.2, 74.2)
- moved D7 23.7 mm to (58.9, 95.5)
- moved G*** 23.7 mm to (67.6, 64.0)
- moved J3 23.7 mm to (73.7, 101.3)
- moved JP2 23.7 mm to (75.7, 99.2)
- moved R11 23.7 mm to (58.9, 98.3)
- moved R12 23.7 mm to (80.3, 69.3)
- moved R13 23.7 mm to (80.3, 72.4)
- moved R4 23.7 mm to (80.3, 75.2)
- moved R7 23.7 mm to (69.8, 83.8)
- moved U1 23.7 mm to (67.5, 74.3)
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Routing:
- net /INT: track 130.6 -> 121.0 mm
- net /DTR: track 79.8 -> 73.8 mm
Other:
- board size 92.5 x 132.6 mm -> 107.7 x 152.4 mm
- board text added: "v-score"
